File: hardware/gate-controller.sch (KiCad schematic (older format))
At the start: 2 parts, among them J1 feather long, J2 feather short

Commit message: Add gate controller circuit components to schematic
Co-Authored-By: Claude Opus 4.6 (1M context) <noreply@anthropic.com>
Parts:
- added C1: 100nF, Capacitor_SMD:C_0805_2012Metric, symbol Device:C
- added J3: Gate_Output, TerminalBlock:TerminalBlock_bornier-2_P5.08mm, symbol Connector:Screw_Terminal_01x02
- added LED1: Green, LED_SMD:LED_0805_2012Metric, symbol Device:LED
- added LED2: WS2812B, LED_SMD:LED_WS2812B_PLCC4_5.0x5.0mm_P3.2mm, symbol LED:WS2812B
- added Q1: 2N3904, Package_TO_SOT_THT:TO-92_Inline, symbol Transistor_BJT:2N3904
- added R1: 1k, Resistor_SMD:R_0805_2012Metric, symbol Device:R
- added R2, R3: 330, Resistor_SMD:R_0805_2012Metric, symbol Device:R
Other:
- note added: "Gate Controller Circuit"
Changed lines of the file:
@@
 Wire Notes Line
 	8350 2550 10500 2550
+Wire Notes Line
+	1500 1200 6500 1200
+Wire Notes Line
+	6500 1200 6500 5500
+Wire Notes Line
+	6500 5500 1500 5500
+Wire Notes Line
+	1500 5500 1500 1200
+Text Notes 1600 1400 0    100  ~ 20
+Gate Controller Circuit
+$Comp
+L Device:R R1
+U 1 1 6651A002
+P 3200 2000
+F 0 "R1" V 3100 2000 50  0000 C CNN
+F 1 "1k" V 3300 2000 50  0000 C CNN
+F 2 "Resistor_SMD:R_0805_2012Metric" H 3200 2000 50  0001 C CNN
+F 3 "~" H 3200 2000 50  0001 C CNN
+	1    3200 2000
+	0    1    1    0
+$EndComp
+$Comp
+L Transistor_BJT:2N3904 Q1
+U 1 1 6651A001
+P 4200 2000
+F 0 "Q1" H 4391 2046 50  0000 L CNN
+F 1 "2N3904" H 4391 1955 50  0000 L CNN
+F 2 "Package_TO_SOT_THT:TO-92_Inline" H 4400 1925 50  0001 L CIN
+F 3 "~" H 4200 2000 50  0001 L CNN
+	1    4200 2000
+	1    0    0    -1
+$EndComp
+$Comp
+L Connector:Screw_Terminal_01x02 J3
+U 1 1 6651A008
+P 5800 1700
+F 0 "J3" H 5880 1692 50  0000 L CNN
+F 1 "Gate_Output" H 5880 1601 50  0000 L CNN
+F 2 "TerminalBlock:TerminalBlock_bornier-2_P5.08mm" H 5800 1700 50  0001 C CNN
+F 3 "~" H 5800 1700 50  0001 C CNN
+	1    5800 1700
+	1    0    0    -1
+$EndComp
+$Comp
+L Device:R R2
+U 1 1 6651A003
+P 2200 3200
+F 0 "R2" H 2270 3246 50  0000 L CNN
+F 1 "330" H 2270 3155 50  0000 L CNN
+F 2 "Resistor_SMD:R_0805_2012Metric" H 2200 3200 50  0001 C CNN
+F 3 "~" H 2200 3200 50  0001 C CNN
+	1    2200 3200
+	1    0    0    -1
+$EndComp
+$Comp
+L Device:LED LED1
+U 1 1 6651A006
+P 2200 3800
+F 0 "LED1" H 2193 4017 50  0000 C CNN
+F 1 "Green" H 2193 3926 50  0000 C CNN
+F 2 "LED_SMD:LED_0805_2012Metric" H 2200 3800 50  0001 C CNN
+F 3 "~" H 2200 3800 50  0001 C CNN
+	1    2200 3800
+	-1   0    0    1
+$EndComp
+$Comp
+L Device:R R3
+U 1 1 6651A004
+P 3200 4600
+F 0 "R3" V 3100 4600 50  0000 C CNN
+F 1 "330" V 3300 4600 50  0000 C CNN
+F 2 "Resistor_SMD:R_0805_2012Metric" H 3200 4600 50  0001 C CNN
+F 3 "~" H 3200 4600 50  0001 C CNN
+	1    3200 4600
+	0    1    1    0
+$EndComp
+$Comp
+L LED:WS2812B LED2
+U 1 1 6651A007
+P 4500 4600
+F 0 "LED2" H 4844 4646 50  0000 L CNN
+F 1 "WS2812B" H 4844 4555 50  0000 L CNN
+F 2 "LED_SMD:LED_WS2812B_PLCC4_5.0x5.0mm_P3.2mm" H 4550 4300 50  0001 L TNN
+F 3 "~" H 4600 4225 50  0001 L TNN
+	1    4500 4600
+	1    0    0    -1
+$EndComp
+$Comp
+L Device:C C1
+U 1 1 6651A005
+P 5500 4600
+F 0 "C1" H 5615 4646 50  0000 L CNN
+F 1 "100nF" H 5615 4555 50  0000 L CNN
+F 2 "Capacitor_SMD:C_0805_2012Metric" H 5538 4450 50  0001 C CNN
+F 3 "~" H 5500 4600 50  0001 C CNN
+	1    5500 4600
+	1    0    0    -1
+$EndComp
+$Comp
+L power:GND #PWR03
+U 1 1 6651A009
+P 4300 2400
+F 0 "#PWR03" H 4300 2150 50  0001 C CNN
+F 1 "GND" H 4305 2227 50  0000 C CNN
+F 2 "" H 4300 2400 50  0001 C CNN
+F 3 "" H 4300 2400 50  0001 C CNN
+	1    4300 2400
+	1    0    0    -1
+$EndComp
+$Comp
+L power:GND #PWR04
+U 1 1 6651A00A
+P 5600 1900
+F 0 "#PWR04" H 5600 1650 50  0001 C CNN
+F 1 "GND" H 5605 1727 50  0000 C CNN
+F 2 "" H 5600 1900 50  0001 C CNN
+F 3 "" H 5600 1900 50  0001 C CNN
+	1    5600 1900
+	1    0    0    -1
+$EndComp
+$Comp
+L power:GND #PWR05
+U 1 1 6651A00B
+P 2200 4100
+F 0 "#PWR05" H 2200 3850 50  0001 C CNN
+F 1 "GND" H 2205 3927 50  0000 C CNN
+F 2 "" H 2200 4100 50  0001 C CNN
+F 3 "" H 2200 4100 50  0001 C CNN
+	1    2200 4100
+	1    0    0    -1
+$EndComp
+$Comp
+L power:GND #PWR06
+U 1 1 6651A00C
+P 4500 5100
+F 0 "#PWR06" H 4500 4850 50  0001 C CNN
+F 1 "GND" H 4505 4927 50  0000 C CNN
+F 2 "" H 4500 5100 50  0001 C CNN
+F 3 "" H 4500 5100 50  0001 C CNN
+	1    4500 5100
+	1    0    0    -1
+$EndComp
+$Comp
+L power:+3.3V #PWR07
+U 1 1 6651A00D
+P 4500 4200
+F 0 "#PWR07" H 4500 4050 50  0001 C CNN
+F 1 "+3.3V" H 4515 4373 50  0000 C CNN
+F 2 "" H 4500 4200 50  0001 C CNN
+F 3 "" H 4500 4200 50  0001 C CNN
+	1    4500 4200
+	1    0    0    -1
+$EndComp
+$Comp
+L power:GND #PWR08
+U 1 1 6651A00E
+P 5500 4900
+F 0 "#PWR08" H 5500 4650 50  0001 C CNN
+F 1 "GND" H 5505 4727 50  0000 C CNN
+F 2 "" H 5500 4900 50  0001 C CNN
+F 3 "" H 5500 4900 50  0001 C CNN
+	1    5500 4900
+	1    0    0    -1
+$EndComp
+$Comp
+L power:+3.3V #PWR09
+U 1 1 6651A00F
+P 5500 4300
+F 0 "#PWR09" H 5500 4150 50  0001 C CNN
+F 1 "+3.3V" H 5515 4473 50  0000 C CNN
+F 2 "" H 5500 4300 50  0001 C CNN
+F 3 "" H 5500 4300 50  0001 C CNN
+	1    5500 4300
+	1    0    0    -1
+$EndComp
 $EndSCHEMATC
