File: hardware/gate-controller.sch (KiCad schematic (older format))
At the start: 10 parts, among them J1 feather long, J2 feather short, J3 Gate_Output, Q1 2N3904

Commit message: Add timed MQTT gate hold and mini breadboard layout
Parts:
- J3: footprint TerminalBlock:TerminalBlock_bornier-2_P5.08mm -> TerminalBlock_Phoenix:TerminalBlock_Phoenix_MKDS-1,5-2-5.08_1x02_P5.08mm_Horizontal
Changed lines of the file:
@@
 F 0 "J3" H 5880 1692 50  0000 L CNN
 F 1 "Gate_Output" H 5880 1601 50  0000 L CNN
-F 2 "TerminalBlock:TerminalBlock_bornier-2_P5.08mm" H 5800 1700 50  0001 C CNN
+F 2 "TerminalBlock_Phoenix:TerminalBlock_Phoenix_MKDS-1,5-2-5.08_1x02_P5.08mm_Horizontal" H 5800 1700 50  0001 C CNN
 F 3 "~" H 5800 1700 50  0001 C CNN
 	1    5800 1700
