File: hardware/gate-controller.kicad_pcb (KiCad board)
At the start: 2 copper layers, 50.8 x 22.9 mm, 6 parts, among them J1 feather long, J2 feather short

Commit message: Add timed MQTT gate hold and mini breadboard layout
Parts:
- added C1: 100nF, Capacitor_SMD:C_0805_2012Metric, F.Cu at (55.0, 34.0)
- added J3: Gate_Output, TerminalBlock_Phoenix:TerminalBlock_Phoenix_MKDS-1,5-2-5.08_1x02_P5.08mm_Horizontal, F.Cu at (62.1, 36.7)
- added LED1: Green, LED_SMD:LED_0805_2012Metric, F.Cu at (55.1, 40.0)
- added LED2: WS2812B, LED_SMD:LED_WS2812B_PLCC4_5.0x5.0mm_P3.2mm, F.Cu at (48.0, 36.6)
- added Q1: 2N3904, Package_TO_SOT_THT:TO-92_Inline, F.Cu at (33.7, 37.0)
- added R1: 1k, Resistor_SMD:R_0805_2012Metric, F.Cu at (41.4, 31.5)
- added R2: 330, Resistor_SMD:R_0805_2012Metric, F.Cu at (41.1, 36.5)
- added R3: 330, Resistor_SMD:R_0805_2012Metric, F.Cu at (41.1, 41.5)
Connections:
- net /~RST renamed /~{RST}
- J1 pad 15: +3V3 -> +3.3V
Other:
- net class Default removed
- board text added: "~{RST}"
- board text removed: "~RST"
